File: kicad/roki/roki.kicad_pcb (KiCad board)
At the start: 2 copper layers, 75 parts, among them SW1 RotaryEncoder_Switch, SW2 SW_SPDT, U1 Nice_Nano_V2

Commit message: feat(kicad): add right side
Parts:
- added BT2: Battery_Cell, Battery:BatteryHolder_MPD_BH-18650-PC2, F.Cu at (161.7, 184.4)
- added D31: Diode, ScottoKeebs_Components:Diode_SOD-123, B.Cu at (277.0, 127.5)
- added D32: Diode, ScottoKeebs_Components:Diode_SOD-123, B.Cu at (432.7, 166.5)
- added D33: Diode, ScottoKeebs_Components:Diode_SOD-123, B.Cu at (426.8, 166.5)
- added D34: Diode, ScottoKeebs_Components:Diode_SOD-123, B.Cu at (421.0, 166.5)
- added D35: Diode, ScottoKeebs_Components:Diode_SOD-123, B.Cu at (415.2, 166.5)
- added D36: Diode, ScottoKeebs_Components:Diode_SOD-123, B.Cu at (409.3, 166.5)
- added D37: Diode, ScottoKeebs_Components:Diode_SOD-123, B.Cu at (277.0, 146.6)
- added D38: Diode, ScottoKeebs_Components:Diode_SOD-123, B.Cu at (432.7, 171.5)
- added D39: Diode, ScottoKeebs_Components:Diode_SOD-123, B.Cu at (426.8, 171.5)
- added D40: Diode, ScottoKeebs_Components:Diode_SOD-123, B.Cu at (421.0, 171.5)
- added D41: Diode, ScottoKeebs_Components:Diode_SOD-123, B.Cu at (415.2, 171.5)
- added D42: Diode, ScottoKeebs_Components:Diode_SOD-123, B.Cu at (409.3, 171.5)
- added D43: Diode, ScottoKeebs_Components:Diode_SOD-123, B.Cu at (277.0, 165.6)
- added D44: Diode, ScottoKeebs_Components:Diode_SOD-123, B.Cu at (432.7, 176.5)
- added D45: Diode, ScottoKeebs_Components:Diode_SOD-123, B.Cu at (426.8, 176.5)
- added D46: Diode, ScottoKeebs_Components:Diode_SOD-123, B.Cu at (421.0, 176.5)
- added D47: Diode, ScottoKeebs_Components:Diode_SOD-123, B.Cu at (415.2, 176.5)
- added D48: Diode, ScottoKeebs_Components:Diode_SOD-123, B.Cu at (409.3, 176.5)
- added D49: Diode, ScottoKeebs_Components:Diode_SOD-123, B.Cu at (277.0, 184.7)
- added D50: Diode, ScottoKeebs_Components:Diode_SOD-123, B.Cu at (432.7, 181.4)
- added D51: Diode, ScottoKeebs_Components:Diode_SOD-123, B.Cu at (426.8, 181.4)
- added D52: Diode, ScottoKeebs_Components:Diode_SOD-123, B.Cu at (421.0, 181.4)
- added D53: Diode, ScottoKeebs_Components:Diode_SOD-123, B.Cu at (415.2, 181.4)
- added D54: Diode, ScottoKeebs_Components:Diode_SOD-123, B.Cu at (409.3, 181.4)
- added D55: Diode, ScottoKeebs_Components:Diode_SOD-123, B.Cu at (430.7, 212.3)
- added D56: Diode, ScottoKeebs_Components:Diode_SOD-123, B.Cu at (425.1, 212.3)
- added D57: Diode, ScottoKeebs_Components:Diode_SOD-123, B.Cu at (419.5, 212.3)
- added D58: Diode, ScottoKeebs_Components:Diode_SOD-123, B.Cu at (413.9, 212.3)
- added D59: Diode, ScottoKeebs_Components:Diode_SOD-123, B.Cu at (408.3, 212.3)
- added D60: Diode, ScottoKeebs_Components:Diode_SOD-123, B.Cu at (402.7, 212.4)
- added S30: Keyswitch, ScottoKeebs_Hotswap:Hotswap_MX_1.00u, F.Cu at (281.9, 133.6)
- added S31: Keyswitch, ScottoKeebs_Hotswap:Hotswap_MX_1.00u, F.Cu at (262.9, 131.6)
- added S32: Keyswitch, ScottoKeebs_Hotswap:Hotswap_MX_1.00u, F.Cu at (243.8, 116.6)
- added S33: Keyswitch, ScottoKeebs_Hotswap:Hotswap_MX_1.00u, F.Cu at (224.8, 111.6)
- added S34: Keyswitch, ScottoKeebs_Hotswap:Hotswap_MX_1.00u, F.Cu at (205.7, 117.6)
- added S35: Keyswitch, ScottoKeebs_Hotswap:Hotswap_MX_1.00u, F.Cu at (186.7, 120.6)
- added S36: Keyswitch, ScottoKeebs_Hotswap:Hotswap_MX_1.00u, F.Cu at (281.9, 152.7)
- added S37: Keyswitch, ScottoKeebs_Hotswap:Hotswap_MX_1.00u, F.Cu at (262.9, 150.7)
- added S38: Keyswitch, ScottoKeebs_Hotswap:Hotswap_MX_1.00u, F.Cu at (243.8, 135.7)
- added S39: Keyswitch, ScottoKeebs_Hotswap:Hotswap_MX_1.00u, F.Cu at (224.8, 130.7)
- added S40: Keyswitch, ScottoKeebs_Hotswap:Hotswap_MX_1.00u, F.Cu at (205.7, 136.7)
- added S41: Keyswitch, ScottoKeebs_Hotswap:Hotswap_MX_1.00u, F.Cu at (186.7, 139.7)
- added S42: Keyswitch, ScottoKeebs_Hotswap:Hotswap_MX_1.00u, F.Cu at (281.9, 171.7)
- added S43: Keyswitch, ScottoKeebs_Hotswap:Hotswap_MX_1.00u, F.Cu at (262.9, 169.7)
- added S44: Keyswitch, ScottoKeebs_Hotswap:Hotswap_MX_1.00u, F.Cu at (243.8, 154.7)
- added S45: Keyswitch, ScottoKeebs_Hotswap:Hotswap_MX_1.00u, F.Cu at (224.8, 149.7)
- added S46: Keyswitch, ScottoKeebs_Hotswap:Hotswap_MX_1.00u, F.Cu at (205.7, 155.7)
- added S47: Keyswitch, ScottoKeebs_Hotswap:Hotswap_MX_1.00u, F.Cu at (186.7, 158.7)
- added S48: Keyswitch, ScottoKeebs_Hotswap:Hotswap_MX_1.00u, F.Cu at (281.9, 190.8)
- added S49: Keyswitch, ScottoKeebs_Hotswap:Hotswap_MX_1.00u, F.Cu at (262.9, 188.8)
- added S50: Keyswitch, ScottoKeebs_Hotswap:Hotswap_MX_1.00u, F.Cu at (243.8, 173.8)
- added S51: Keyswitch, ScottoKeebs_Hotswap:Hotswap_MX_1.00u, F.Cu at (224.8, 168.8)
- added S52: Keyswitch, ScottoKeebs_Hotswap:Hotswap_MX_1.00u, F.Cu at (205.7, 174.8)
- added S53: Keyswitch, ScottoKeebs_Hotswap:Hotswap_MX_1.00u, F.Cu at (186.7, 177.8)
- added S54: Keyswitch, ScottoKeebs_Hotswap:Hotswap_MX_1.00u, F.Cu at (291.0, 246.9)
- added S55: Keyswitch, ScottoKeebs_Hotswap:Hotswap_MX_1.00u, F.Cu at (275.5, 246.9)
- added S56: Keyswitch, ScottoKeebs_Hotswap:Hotswap_MX_1.00u, F.Cu at (259.9, 246.9)
- added S57: Keyswitch, ScottoKeebs_Hotswap:Hotswap_MX_1.00u, F.Cu at (244.4, 246.9)
- added S58: Keyswitch, ScottoKeebs_Hotswap:Hotswap_MX_1.00u, F.Cu at (228.8, 246.9)
- added SW3: RotaryEncoder_Switch, Rotary_Encoder:RotaryEncoder_Alps_EC11E-Switch_Vertical_H20mm, F.Cu at (444.6, 207.4)
- added SW4: SW_SPDT, Button_Switch_SMD:SW_SPDT_PCM12, F.Cu at (447.5, 220.5)
- added U3: ~, Library:thumb_stick, F.Cu at (515.0, 192.4)
- added U4: Nice_Nano_V2, ScottoKeebs_MCU:Nice_Nano_V2, F.Cu at (452.1, 129.6)
- moved REF** 10.1 mm to (1.27, 109.1)
- moved REF** 10.1 mm to (50.4, 103.4)
- moved D24 9.45 mm to (64.2, 168.7)
- moved S22 9.45 mm to (34.0, 165.8)
- moved D19 9.45 mm to (-31.0, 181.7)
- moved D20 9.45 mm to (-12.0, 179.7)
- moved D21 9.45 mm to (7.08, 164.7)
- moved D22 9.45 mm to (26.1, 159.7)
- moved S19 9.45 mm to (-23.1, 187.8)
- moved S20 9.45 mm to (-4.07, 185.8)
- moved S21 9.45 mm to (15.0, 170.8)
- moved D23 9.45 mm to (45.2, 165.7)
- moved S23 9.45 mm to (53.1, 171.8)
- moved S24 9.45 mm to (72.1, 174.8)
- moved D18 9.45 mm to (64.2, 149.6)
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Connections:
- U1 pad 1: Net-(SW2-C) -> unconnected-(U1-Pad1)
- U1 pad 23: unconnected-(U1-GND-Pad23) -> Net-(SW2-C)
- U2 pad 1: AY -> GND
- U2 pad 2: VCC -> AX
- U2 pad 3: GND -> VCC
- U2 pad 4: AX -> GND
- U2 pad 5: VCC -> AY
- U2 pad 6: GND -> VCC
- U2 pad 7: GND -> SS
- U2 pad 8: SS -> GND

Commit message: feat(kicad): update pcb
Parts:
- removed the REF** at (50.4, 103.4)
- added BZ1: Buzzer, Buzzer_Beeper:Buzzer_TDK_PS1240P02BT_D12.2mm_H6.5mm, F.Cu at (119.2, 110.1)
- added BZ2: Buzzer, Buzzer_Beeper:Buzzer_TDK_PS1240P02BT_D12.2mm_H6.5mm, F.Cu at (195.2, 110.1)
- added REF**: MountingHole_3.2mm_M3, MountingHole:MountingHole_3.2mm_M3, F.Cu at (350.4, 159.2)
- added REF**: MountingHole_3.2mm_M3, MountingHole:MountingHole_3.2mm_M3, F.Cu at (170.2, 185.5)
- added REF**: MountingHole_3.2mm_M3, MountingHole:MountingHole_3.2mm_M3, F.Cu at (312.9, 115.1)
- added REF**: MountingHole_3.2mm_M3, MountingHole:MountingHole_3.2mm_M3, F.Cu at (207.4, 139.4)
- added REF**: MountingHole_3.2mm_M3, MountingHole:MountingHole_3.2mm_M3, F.Cu at (302.9, 198.7)
- added REF**: MountingHole_3.2mm_M3, MountingHole:MountingHole_3.2mm_M3, F.Cu at (192.2, 132.1)
- added REF**: MountingHole_3.2mm_M3, MountingHole:MountingHole_3.2mm_M3, F.Cu at (192.2, 164.6)
- added REF**: MountingHole_3.2mm_M3, MountingHole:MountingHole_3.2mm_M3, F.Cu at (192.2, 99.6)
- added REF**: MountingHole_3.2mm_M3, MountingHole:MountingHole_3.2mm_M3, F.Cu at (232.7, 102.5)
- added REF**: MountingHole_3.2mm_M3, MountingHole:MountingHole_3.2mm_M3, F.Cu at (107.0, 139.4)
- SW2, SW4: moved to B.Cu
- moved U3 329.4 mm to (185.6, 199.0), turned to -135 degrees
- moved U4 235.9 mm to (216.5, 116.9)
- moved SW4 234.2 mm to (246.1, 101.2)
- moved SW3 226.8 mm to (220.7, 171.3), turned to -90 degrees
- moved D59 208.2 mm to (200.5, 225.1), turned to 45 degrees
- moved D58 196.4 mm to (217.5, 209.4), turned to 30 degrees
- moved D60 187.5 mm to (218.2, 178.8), turned to -90 degrees
- moved D36 183.5 mm to (234.3, 111.5)
- moved D57 182.1 mm to (237.9, 198.7), turned to 15 degrees
- moved D42 179.8 mm to (234.3, 130.6)
- moved D48 177.1 mm to (234.3, 149.6)
- moved D54 175.5 mm to (234.3, 168.7)
- moved D35 171.9 mm to (253.3, 108.5)
- moved D41 167.7 mm to (253.3, 127.6)
- moved D56 165.7 mm to (260.4, 193.7)
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Connections:
- SW4 pad 1: unconnected-(SW4-A-Pad1) -> Net-(SW4-A)
- SW4 pad 3: Net-(SW4-C) -> unconnected-(SW4-C-Pad3)
- U1 pad 1: unconnected-(U1-Pad1) -> BUZZ
- U4 pad 1: unconnected-(U4-Pad1) -> BUZZR
- U4 pad 23: Net-(SW4-C) -> Net-(SW4-A)
Other:
- board outline added: 144.9 x 130 mm

Commit message: feat(kicad): pin components
Parts:
- removed the REF** at (120.8, 217.9)
- removed the REF** at (39.9, 179.1)
- removed the REF** at (207.4, 139.4)
- added REF**: MountingHole_3.2mm_M3, MountingHole:MountingHole_3.2mm_M3, F.Cu at (101.7, 202.3)
- added REF** (x2): MountingHole_3.2mm_M3, MountingHole:MountingHole_3.2mm_M3, F.Cu at (207.4, 139.4)
- added REF**: MountingHole_3.2mm_M3, MountingHole:MountingHole_3.2mm_M3, F.Cu at (39.6, 181.3)
- added REF**: MountingHole_3.2mm_M3, MountingHole:MountingHole_3.2mm_M3, F.Cu at (212.7, 202.3)
- added REF**: MountingHole_3.2mm_M3, MountingHole:MountingHole_3.2mm_M3, F.Cu at (274.8, 181.3)
Connections:
- BZ1 pad 1: (no net) -> BUZZ
- BZ1 pad 2: (no net) -> GND
- BZ2 pad 1: (no net) -> BUZZR
- BZ2 pad 2: (no net) -> GNDR

Commit message: feat(kicad): update files
Parts:
- removed the REF** at (207.4, 139.4)
- moved D30 5.00 mm to (99.1, 174.8)
- moved D60 5.00 mm to (215.2, 174.8)
- moved SW1 5.00 mm to (101.6, 167.3)
- moved SW3 5.00 mm to (217.7, 167.3)
- moved REF** 1.00 mm to (171.2, 185.5)
- moved REF** 1.00 mm to (143.2, 185.5)
Routing:
- net Col 1: track 0.00 -> 275.9 mm, vias 0 -> 1
- net Col 2: track 0.00 -> 233.0 mm, vias 0 -> 3
- net Col 5: track 0.00 -> 229.3 mm, vias 0 -> 1
- net Row 3: track 0.00 -> 227.5 mm, vias 0 -> 10
- net Col 4: track 0.00 -> 227.2 mm, vias 0 -> 1
- net Col 3: track 0.00 -> 226.0 mm, vias 0 -> 3
- net Row 5: track 0.00 -> 204.4 mm
- net Row 4: track 0.00 -> 197.9 mm, vias 0 -> 7
- net Row 2: track 0.00 -> 195.7 mm, vias 0 -> 10
- net SS: track 0.00 -> 194.5 mm
- net GND: track 0.00 -> 191.9 mm
- net Row 1: track 0.00 -> 179.1 mm, vias 0 -> 10
- net Col 6: track 0.00 -> 144.0 mm
- net Net-(BT1--): track 0.00 -> 123.2 mm
- net VCC: track 0.00 -> 113.0 mm
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Other:
- board size 144.9 x 130 mm -> 393.5 x 142.2 mm

Commit message: feat(kicad): update pcb
Parts:
- added REF**: MountingHole_3.2mm_M3, MountingHole:MountingHole_3.2mm_M3, F.Cu at (226.9, 231.3)
- added REF**: MountingHole_3.2mm_M3, MountingHole:MountingHole_3.2mm_M3, F.Cu at (130.0, 220.1)
- added REF**: MountingHole_3.2mm_M3, MountingHole:MountingHole_3.2mm_M3, F.Cu at (184.3, 220.1)
- added REF**: MountingHole_3.2mm_M3, MountingHole:MountingHole_3.2mm_M3, F.Cu at (87.5, 231.3)
- moved REF** 7.00 mm to (171.2, 178.5)
- moved REF** 7.00 mm to (143.2, 178.5)
- moved REF** 4.63 mm to (104.0, 206.3)
- moved REF** 4.63 mm to (210.3, 206.3)
- moved REF** 1.50 mm to (13.0, 198.7)
- moved REF** 1.50 mm to (301.4, 198.7)
- moved SW2 1.50 mm to (68.3, 102.7)
- moved SW4 1.50 mm to (246.1, 102.7)
- moved U1 0.80 mm to (97.8, 117.7)
- moved U4 0.80 mm to (216.5, 117.7)
Connections:
- D32 pad 1: Col 1R -> Col 2R
- D33 pad 1: Col 1R -> Col 3R
- D34 pad 1: Col 1R -> Col 4R
- D35 pad 1: Col 1R -> Col 5R
- D36 pad 1: Col 2R -> Col 6R
- D37 pad 1: Col 2R -> Col 1R
- D39 pad 1: Col 2R -> Col 3R
- D40 pad 1: Col 2R -> Col 4R
- D41 pad 1: Col 3R -> Col 5R
- D42 pad 1: Col 3R -> Col 6R
- D43 pad 1: Col 3R -> Col 1R
- D44 pad 1: Col 3R -> Col 2R
- D47 pad 1: Col 4R -> Col 5R
- D48 pad 1: Col 4R -> Col 6R
- D49 pad 1: Col 4R -> Col 1R
- D50 pad 1: Col 4R -> Col 2R
- D51 pad 1: Col 5R -> Col 3R
- D52 pad 1: Col 5R -> Col 4R
- D54 pad 1: Col 5R -> Col 6R
- D55 pad 1: Col 5R -> Col 1R
- D56 pad 1: Col 6R -> Col 2R
- D57 pad 1: Col 6R -> Col 3R
- D58 pad 1: Col 6R -> Col 4R
- D59 pad 1: Col 6R -> Col 5R
- S31 pad 1: Row 2R -> Row 1R
- S32 pad 1: Row 3R -> Row 1R
- S33 pad 1: Row 4R -> Row 1R
- S34 pad 1: Row 5R -> Row 1R
- S37 pad 1: Row 3R -> Row 2R
- S38 pad 1: Row 4R -> Row 2R
- S39 pad 1: Row 5R -> Row 2R
- S40 pad 1: Row 1R -> Row 2R
- S43 pad 1: Row 4R -> Row 3R
- S44 pad 1: Row 5R -> Row 3R
- S45 pad 1: Row 1R -> Row 3R
- S46 pad 1: Row 2R -> Row 3R
- S49 pad 1: Row 5R -> Row 4R
- S50 pad 1: Row 1R -> Row 4R
- S51 pad 1: Row 2R -> Row 4R
- S52 pad 1: Row 3R -> Row 4R
- S55 pad 1: Row 1R -> Row 5R
- S56 pad 1: Row 2R -> Row 5R
- S57 pad 1: Row 3R -> Row 5R
- S58 pad 1: Row 4R -> Row 5R
Routing:
- net Col 1R: track 0.00 -> 245.2 mm
- net Row 4R: track 0.00 -> 228.2 mm, vias 0 -> 6
- net Col 2R: track 0.00 -> 221.9 mm
- net Col 3R: track 0.00 -> 212.1 mm
- net Row 3R: track 0.00 -> 211.4 mm, vias 0 -> 6
- net Col 4R: track 0.00 -> 207.2 mm
- net Row 2R: track 0.00 -> 198.9 mm, vias 0 -> 6
- net Row 1R: track 0.00 -> 192.0 mm, vias 0 -> 6
- net Col 5R: track 0.00 -> 189.5 mm
- net Row 5R: track 0.00 -> 183.0 mm, vias 0 -> 2
- net GNDR: track 0.00 -> 153.9 mm
- net Net-(BT2--): track 0.00 -> 131.6 mm, vias 0 -> 1
- net VCCR: track 0.00 -> 120.1 mm
- net AYR: track 0.00 -> 114.0 mm
- net AXR: track 0.00 -> 107.9 mm
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Other:
- board size 393.5 x 142.2 mm -> 393.6 x 142.2 mm
